File: v2.1/power-switch (ds lite)/power-switch.kicad_pcb (KiCad board)
At the start: 2 copper layers, 19 x 6.8 mm, 6 parts

Commit message: consistify labels
Parts:
- removed the REF** at (105.5, 67.3)
Connections:
- REF** pad 1: (no net) -> GND
Routing:
- net GND: vias 0 -> 2
Other:
- board text added: "2"
- board text added: "C"
- board text added: "SW-C"
- board text removed: "B+"
- board text removed: "PWR IN"
- board text removed: "SW C"
- board text removed: "SW ON"
