File: v2.1/Momentary-Power-Toggle.sch (KiCad schematic (older format))
At the start: 13 parts, among them J1 PWR_C, J2 PWR_2, J3 BTN, J4 GND, Q1 IRF7317PbF

Commit message: cleanup
cleaned up readme, board files, added renders, made small tweaks to some of the boards (added identifiers and changed labels for consistency)
Parts:
- Q1: symbol misc:IRF7317PbF -> Momentary-Power-Toggle-rescue:IRF7317PbF-misc
Changed lines of the file:
@@
 $EndComp
 $Comp
-L misc:IRF7317PbF Q1
+L Momentary-Power-Toggle-rescue:IRF7317PbF-misc Q1
 U 1 1 5F3FED7F
 P 6000 3300
@@
 	4450 2700 4450 3050
 $Comp
-L power:GND #PWR?
+L power:GND #PWR0101
 U 1 1 5F68BE7D
 P 2250 3450
-F 0 "#PWR?" H 2250 3200 50  0001 C CNN
+F 0 "#PWR0101" H 2250 3200 50  0001 C CNN
 F 1 "GND" H 2255 3277 50  0000 C CNN
 F 2 "" H 2250 3450 50  0001 C CNN
